File: hardware/super-mini-mesh-kicad/super-mini-mesh-kicad.kicad_sch (KiCad schematic)
At the start: 4 parts, among them P1 USB_C_Plug_USB2.0, U1 Wio-SX1262, U2 nice_nano, U3 ssd1306

Commit message: update
Parts:
- removed P1: USB_C_Plug_USB2.0, Connector_USB:USB_C_Plug_Molex_105444, symbol Connector:USB_C_Plug_USB2.0
- removed U1: Wio-SX1262, wio-sx1262:wio-sx1262, symbol ProLib_pcs_2024-10-14:libdb_Module/114993390
- removed U2: nice_nano, footprints:nice_nano, symbol nice_nano:nice_nano
- removed U3: ssd1306, footprints:ssd1306_a, symbol picoco2:ssd1306
- added J1: Conn_01x02_Socket, Connector_JST:JST_PH_B2B-PH-K_1x02_P2.00mm_Vertical, symbol Connector:Conn_01x02_Socket
- added J2, J3: Conn_01x04_Pin, Connector_PinHeader_2.54mm:PinHeader_1x04_P2.54mm_Vertical, symbol Connector:Conn_01x04_Pin
- added J4: Conn_01x01_Socket, Connector_PinSocket_2.54mm:PinSocket_1x01_P2.54mm_Vertical, symbol Connector:Conn_01x01_Socket
- added R1, R2: R, Resistor_THT:R_Axial_DIN0204_L3.6mm_D1.6mm_P1.90mm_Vertical, symbol Device:R
- added SW1: SW_Push, Button_Switch_THT:SW_PUSH_6mm, symbol Switch:SW_Push
- added U1: wio-sx1262, wio-sx1262:wio-sx1262, symbol sweet-p:wio-sx1262
- added U2: nice_nano_clean, footprints:nice_nano_cleanest, symbol nice_nano:nice_nano_clean
Connections:
- new net 3V3: J2.1 (Pin_1), J3.2 (Pin_2), U1.8 (VCC), U2.21 (VCC)
- new net ANT: J4.1 (Pin_1), U1.9 (ANT)
- new net BAT: J1.1 (Pin_1), R2.1, U2.24 (BAT), U2.25 (BAT)
- new net BATT_MEASURE: R1.1, R2.2, U2.20 (AIN7/P0.31)
- new net BUSY: U1.11 (BUSY), U2.19 (AIN5/P0.29)
- new net CS: U1.6 (NSS), U2.16 (P1.13)
- new net DIO1: U1.12 (DIO1), U2.14 (NFC2/P0.10)
- new net GND: J1.2 (Pin_2), J2.4 (Pin_4), J3.1 (Pin_1), R1.2, SW1.2, U1.10 (GND2), U1.7 (GND1), U2.23 (GND), U2.26 (GND), U2.3 (GND), U2.4 (GND)
- new net GPS_RX: J2.2 (Pin_2), U2.6 (P0.20)
- new net GPS_TX: J2.3 (Pin_3), U2.7 (P0.22)
- new net LORA_RST: U1.5 (RST), U2.13 (NFC1/P0.09)
- new net MICRO_RST: SW1.1, U2.22 (RST)
- new net MISO: U1.2 (MISO), U2.18 (AIN0/P0.02)
- new net MOSI: U1.3 (MOSI), U2.17 (P1.15)
- new net RF_SW1: U1.1 (RF_SW1)
- new net SCK: U1.4 (SCK), U2.15 (P1.11)
- new net SCL: J3.3 (Pin_3), U2.10 (P0.11)
- new net SDA: J3.4 (Pin_4), U2.11 (P1.04)
