File: hardware/super-mini-mesh-kicad/super-mini-mesh-kicad.kicad_pcb (KiCad board)
At the start: 2 copper layers, 33.5 x 28.5 mm, 4 parts, among them P1 USB_C_Plug_USB2.0, U1 Wio-SX1262, U2 nice_nano, U3 ssd1306

Commit message: update
Parts:
- removed P1: USB_C_Plug_USB2.0, Connector_USB:USB_C_Plug_Molex_105444
- removed U3: ssd1306, footprints:ssd1306_a
- added J1: Conn_01x02_Socket, Connector_JST:JST_PH_B2B-PH-K_1x02_P2.00mm_Vertical, F.Cu at (106.7, 28.4)
- added J2: Conn_01x04_Pin, Connector_PinHeader_2.54mm:PinHeader_1x04_P2.54mm_Vertical, B.Cu at (80.7, 25.5)
- added J3: Conn_01x04_Pin, Connector_PinHeader_2.54mm:PinHeader_1x04_P2.54mm_Vertical, F.Cu at (84.6, 25.5)
- added J4: Conn_01x01_Socket, Connector_PinSocket_2.54mm:PinSocket_1x01_P2.54mm_Vertical, F.Cu at (107.6, 41.6)
- added R1: R, Resistor_THT:R_Axial_DIN0204_L3.6mm_D1.6mm_P1.90mm_Vertical, F.Cu at (66.8, 27.5)
- added R2: R, Resistor_THT:R_Axial_DIN0204_L3.6mm_D1.6mm_P1.90mm_Vertical, F.Cu at (61.4, 27.5)
- added SW1: SW_Push, Button_Switch_THT:SW_PUSH_6mm, F.Cu at (96.6, 32.8)
- U1: value Wio-SX1262 -> wio-sx1262; moved to F.Cu
- U2: value nice_nano -> nice_nano_clean; footprint footprints:nice_nano -> footprints:nice_nano_cleanest
- moved U2 50.7 mm to (77.5, 38.3)
- moved U1 31.3 mm to (95.1, 35.2), turned to -90 degrees
Connections:
- U1 pad 1: unconnected-(U1-RF_SW1-Pad1) -> RF_SW1
- U1 pad 10: unconnected-(U1-GND2-Pad10) -> GND
- U1 pad 11: unconnected-(U1-BUSY-Pad11) -> BUSY
- U1 pad 12: unconnected-(U1-DIO1-Pad12) -> DIO1
- U1 pad 2: unconnected-(U1-MISO-Pad2) -> MISO
- U1 pad 3: unconnected-(U1-MOSI-Pad3) -> MOSI
- U1 pad 4: unconnected-(U1-SCK-Pad4) -> SCK
- U1 pad 5: unconnected-(U1-RST-Pad5) -> LORA_RST
- U1 pad 6: unconnected-(U1-NSS-Pad6) -> CS
- U1 pad 7: unconnected-(U1-GND1-Pad7) -> GND
- U1 pad 8: unconnected-(U1-VCC-Pad8) -> 3V3
- U1 pad 9: unconnected-(U1-ANT-Pad9) -> ANT
- U2 pad 10: unconnected-(U2-P0.11-Pad10) -> SCL
- U2 pad 11: unconnected-(U2-P1.04-Pad11) -> SDA
- U2 pad 13: unconnected-(U2-NFC1/P0.09-Pad13) -> LORA_RST
- U2 pad 14: unconnected-(U2-NFC2/P0.10-Pad14) -> DIO1
- U2 pad 15: unconnected-(U2-P1.11-Pad15) -> SCK
- U2 pad 16: unconnected-(U2-P1.13-Pad16) -> CS
- U2 pad 17: unconnected-(U2-P1.15-Pad17) -> MOSI
- U2 pad 18: unconnected-(U2-AIN0/P0.02-Pad18) -> MISO
- U2 pad 19: unconnected-(U2-AIN5/P0.29-Pad19) -> BUSY
- U2 pad 20: unconnected-(U2-AIN7/P0.31-Pad20) -> BATT_MEASURE
- U2 pad 21: unconnected-(U2-VCC-Pad21) -> 3V3
- U2 pad 22: unconnected-(U2-RST-Pad22) -> MICRO_RST
- U2 pad 23: unconnected-(U2-GND-Pad23) -> GND
- U2 pad 24: unconnected-(U2-BATIN/P0.04-Pad24) -> BAT
- U2 pad 3: unconnected-(U2-GND-Pad3) -> GND
- U2 pad 4: unconnected-(U2-GND-Pad4) -> GND
- U2 pad 6: unconnected-(U2-P0.20-Pad6) -> GPS_RX
- U2 pad 7: unconnected-(U2-P0.22-Pad7) -> GPS_TX
Routing:
- net GND: track 0.00 -> 111.4 mm, vias 0 -> 11
- net GPS_TX: track 0.00 -> 70.5 mm, vias 0 -> 4
- net 3V3: track 0.00 -> 62.9 mm, vias 0 -> 5
- net GPS_RX: track 0.00 -> 60.5 mm, vias 0 -> 5
- net BAT: track 0.00 -> 59.6 mm, vias 0 -> 3
- net BUSY: track 0.00 -> 37.5 mm, vias 0 -> 4
- net SDA: track 0.00 -> 36.6 mm, vias 0 -> 3
- net MICRO_RST: track 0.00 -> 36.5 mm, vias 0 -> 1
- net SCL: track 0.00 -> 31.4 mm, vias 0 -> 3
- net MISO: track 0.00 -> 23.5 mm, vias 0 -> 2
- net DIO1: track 0.00 -> 23.1 mm, vias 0 -> 4
- net CS: track 0.00 -> 22.8 mm, vias 0 -> 2
- net MOSI: track 0.00 -> 22.2 mm, vias 0 -> 2
- net SCK: track 0.00 -> 18.3 mm, vias 0 -> 2
- net LORA_RST: track 0.00 -> 14.6 mm, vias 0 -> 2
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Other:
- board size 33.5 x 28.5 mm -> 51.9 x 23.2 mm
- board text added: "20"
- board text added: "22"
- board text added: "3V"
- board text added: "ANT"
- board text added: "BAT"
- board text added: "GND"
- board text added: "RST"
- board text added: "SCL"
- board text added: "SDA"
- board text added: "v0.1"
- board text added: "waterbearfieldschool.org/thistle"

Commit message: update
Parts:
- moved J4 0.73 mm to (107.8, 42.3)
Other:
- board text added: "ANTENNA"
- board text removed: "ANT"
Changed lines of the file:
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@@
 		)
 		(fp_text user "${REFERENCE}"
-			(at 0 3.81 360)
+			(at 0 3.81 0)
 			(layer "F.Fab")
 			(effects
@@
 	(footprint "Connector_PinSocket_2.54mm:PinSocket_1x01_P2.54mm_Vertical"
 		(layer "F.Cu")
-		(at 107.6 41.6)
+		(at 107.8 42.3)
 		(descr "Through hole straight socket strip, 1x01, 2.54mm pitch, single row (from Kicad 4.0.7), script generated")
 		(tags "Through hole socket strip THT 1x01 2.54mm single row")
@@
 	)
 	(gr_text "waterbearfieldschool.org/thistle"
-		(at 110.9 45.1 90)
+		(at 110.8 45.7 90)
 		(layer "F.SilkS")
 		(effects
@@
 		)
 	)
-	(gr_text "ANT"
-		(at 106.7 40.1 0)
+	(gr_text "ANTENNA"
+		(at 108.25 40.7 90)
 		(layer "F.SilkS")
 		(effects
@@
 	)
 	(gr_text "v0.1"
-		(at 107.2 46 0)
+		(at 107.1 47 0)
 		(layer "F.SilkS")
 		(effects
@@
 	)
 	(segment
+		(start 107.1 41.6)
+		(end 107.8 42.3)
+		(width 0.7)
+		(layer "F.Cu")
+		(net 16)
+	)
+	(segment
 		(start 105.8 41.6)
-		(end 107.6 41.6)
-		(width 0.7)
-		(layer "F.Cu")
+		(end 107.1 41.6)
+		(width 0.7)
+		(layer "F.Cu")
